File: telemetry_box_01/telemetry_box_01.kicad_sch (KiCad schematic)
At the start: 103 parts, among them J1 78646-3001, J2 U.FL-R-SMT-1_10_, J3 U.FL-R-SMT-1_10_, J4 12401832E402A, U1 nRF52840, U2 A9G, U3 STBC08PMR, U4 TPS7A2633DRVR, Y1 Crystal_GND24, Y2 ABS04W-32.768KHZ-4-D2-T5

Commit message: fix(vias): blind vias have been removed to optimize production
Connections:
- net NRF_GPIO_01: now also U1.A10 (AIN5/P0.29); no longer U1.B11 (AIN4/P0.28)
- net NRF_GPIO_02: now also U1.A8 (AIN7/P0.31); no longer U1.B9 (AIN6/P0.30)
- net NRF_RESET: now also U1.AC15 (P0.19), U1.AC17 (P0.21), U1.AC19 (P0.23), U1.AC21 (P0.25)
Other:
- note added: "TODO: Посчитать ёмкости на кварцах Добавить светодиоды Добавить тестовые площадки Добавить разъём swd Добавить разъём uart дополнительный Добавить gpio"
- note removed: "TODO: +Посчитать ёмкости на кварцах +Добавить светодиоды +Добавить тестовые площадки +Добавить разъём swd +Добавить разъём uart дополнительный +Добавить gpio"
- note removed: "Проектирование антенны BLE: https://e2e.ti.com/support/wireless-connectivity/wi-fi-group/wifi/f/wi-fi-forum/730866/cc3200mod-want-cad-altium-file https://e2e.ti.com/support/wireless-connectivity/wi-fi-group/wifi/f/wi-fi-forum/572489/cc3100mod-antenna-s-transmission-line-mismatch"
Changed lines of the file:
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@@
   (junction (at 490.22 355.6) (diameter 0) (color 0 0 0 0)
   )
+  (junction (at 214.63 184.15) (diameter 0) (color 0 0 0 0)
+  )
   (junction (at 262.89 292.1) (diameter 0) (color 0 0 0 0)
   )
@@
   (junction (at 377.19 318.77) (diameter 0) (color 0 0 0 0)
   )
+  (junction (at 214.63 194.31) (diameter 0) (color 0 0 0 0)
+  )
   (junction (at 587.59 259.03) (diameter 0) (color 0 0 0 0)
   )
@@
   (junction (at 476.25 203.2) (diameter 0) (color 0 0 0 0)
   )
+  (junction (at 214.63 189.23) (diameter 0) (color 0 0 0 0)
+  )
   (junction (at 403.86 308.61) (diameter 0) (color 0 0 0 0)
   )
@@
     (stroke (width 0) (type default))
   )
+  (wire (pts (xy 198.12 209.55) (xy 200.66 209.55))
+    (stroke (width 0) (type default))
+  )
   (wire (pts (xy 88.9 328.93) (xy 92.71 328.93))
     (stroke (width 0) (type default))
@@
     (stroke (width 0) (type default))
   )
-  (wire (pts (xy 198.12 207.01) (xy 200.66 207.01))
-    (stroke (width 0) (type default))
-  )
   (wire (pts (xy 462.28 308.61) (xy 462.28 311.15))
     (stroke (width 0) (type default))
@@
     (stroke (width 0) (type default))
   )
+  (wire (pts (xy 198.12 199.39) (xy 214.63 199.39))
+    (stroke (width 0) (type default))
+  )
   (wire (pts (xy 641.35 86.36) (xy 643.89 86.36))
     (stroke (width 0) (type default))
@@
     (stroke (width 0) (type default))
   )
+  (wire (pts (xy 198.12 184.15) (xy 214.63 184.15))
+    (stroke (width 0) (type default))
+  )
   (wire (pts (xy 307.34 374.65) (xy 347.98 374.65))
     (stroke (width 0) (type default))
@@
     (stroke (width 0) (type default))
   )
-  (wire (pts (xy 198.12 212.09) (xy 200.66 212.09))
-    (stroke (width 0) (type default))
-  )
   (wire (pts (xy 262.89 303.53) (xy 269.24 303.53))
     (stroke (width 0) (type default))
@@
     (stroke (width 0) (type default))
   )
+  (wire (pts (xy 198.12 189.23) (xy 214.63 189.23))
+    (stroke (width 0) (type default))
+  )
   (wire (pts (xy 542.29 68.58) (xy 542.29 66.04))
     (stroke (width 0) (type default))
@@
     (stroke (width 0) (type default))
   )
+  (wire (pts (xy 214.63 189.23) (xy 214.63 184.15))
+    (stroke (width 0) (type default))
+  )
   (wire (pts (xy 516.47 193.2) (xy 513.45 193.2))
     (stroke (width 0) (type default))
@@
     (stroke (width 0) (type default))
   )
+  (wire (pts (xy 214.63 199.39) (xy 214.63 194.31))
+    (stroke (width 0) (type default))
+  )
   (wire (pts (xy 566 181.56) (xy 554.57 181.56))
     (stroke (width 0) (type default))
@@
     (stroke (width 0) (type default))
   )
+  (wire (pts (xy 214.63 194.31) (xy 214.63 189.23))
+    (stroke (width 0) (type default))
+  )
   (wire (pts (xy 198.12 138.43) (xy 256.54 138.43))
     (stroke (width 0) (type default))
@@
     (stroke (width 0) (type default))
   )
+  (wire (pts (xy 198.12 194.31) (xy 214.63 194.31))
+    (stroke (width 0) (type default))
+  )
   (wire (pts (xy 347.98 406.4) (xy 347.98 417.83))
     (stroke (width 0) (type default))
@@
     (stroke (width 0) (type default))
   )
+  (wire (pts (xy 198.12 214.63) (xy 200.66 214.63))
+    (stroke (width 0) (type default))
+  )
   (wire (pts (xy 186.69 50.8) (xy 186.69 53.34))
     (stroke (width 0) (type default))
@@
   )
   (wire (pts (xy 557.53 208.28) (xy 557.53 209.2))
+    (stroke (width 0) (type default))
+  )
+  (wire (pts (xy 214.63 184.15) (xy 217.17 184.15))
     (stroke (width 0) (type default))
   )
@@
     (effects (font (size 1.27 1.27)) (justify left bottom))
   )
-  (text "Проектирование антенны BLE:\nhttps://e2e.ti.com/support/wireless-connectivity/wi-fi-group/wifi/f/wi-fi-forum/730866/cc3200mod-want-cad-altium-file\nhttps://e2e.ti.com/support/wireless-connectivity/wi-fi-group/wifi/f/wi-fi-forum/572489/cc3100mod-antenna-s-transmission-line-mismatch\n\n\n"
-    (at 669.29 378.46 0)
-    (effects (font (size 1.27 1.27)) (justify left bottom))
-  )
   (text "Main power input for every pins\nCap description" (at 172.72 33.02 0)
     (effects (font (size 1.27 1.27)) (justify left bottom))
@@
     (effects (font (size 1.27 1.27)) (justify left bottom))
   )
-  (text "TODO:\n+Посчитать ёмкости на кварцах\n+Добавить светодиоды\n+Добавить тестовые площадки\n+Добавить разъём swd\n+Добавить разъём uart дополнительный\n+Добавить gpio"
+  (text "TODO:\nПосчитать ёмкости на кварцах\nДобавить светодиоды\nДобавить тестовые площадки\nДобавить разъём swd\nДобавить разъём uart дополнительный\nДобавить gpio"
     (at 854.71 45.72 0)
     (effects (font (size 1.27 1.27)) (justify left bottom))
@@
     )
   )
+  (global_label "NRF_RESET" (shape input) (at 217.17 184.15 0) (fields_autoplaced)
+    (effects (font (size 1.27 1.27)) (justify left))
+    (property "Intersheetrefs" "${INTERSHEET_REFS}" (at 230.4776 184.15 0)
+      (effects (font (size 1.27 1.27)) (justify left) hide)
+    )
+  )
   (global_label "A9G_GPS_ANT" (shape input) (at 566.42 208.28 0) (fields_autoplaced)
     (effects (font (size 1.27 1.27)) (justify left))
@@
     )
   )
-  (global_label "NRF_GPIO_02" (shape input) (at 200.66 212.09 0) (fields_autoplaced)
-    (effects (font (size 1.27 1.27)) (justify left))
-    (property "Intersheetrefs" "${INTERSHEET_REFS}" (at 216.1638 212.09 0)
+  (global_label "NRF_GPIO_02" (shape input) (at 200.66 214.63 0) (fields_autoplaced)
+    (effects (font (size 1.27 1.27)) (justify left))
+    (property "Intersheetrefs" "${INTERSHEET_REFS}" (at 216.1638 214.63 0)
       (effects (font (size 1.27 1.27)) (justify left) hide)
     )
@@
     )
   )
-  (global_label "NRF_GPIO_01" (shape input) (at 200.66 207.01 0) (fields_autoplaced)
-    (effects (font (size 1.27 1.27)) (justify left))
-    (property "Intersheetrefs" "${INTERSHEET_REFS}" (at 216.1638 207.01 0)
-      (effects (font (size 1.27 1.27)) (justify left) hide)
-    )
+  (global_label "NRF_GPIO_01" (shape input) (at 200.66 209.55 0) (fields_autoplaced)
+    (effects (font (size 1.27 1.27)) (justify left))
+    (property "Intersheetrefs" "${INTERSHEET_REFS}" (at 216.1638 209.55 0)
+      (effects (font (size 1.27 1.27)) (justify left) hide)
+    )

Commit message: feat(board): optimization of component placement -reduce product dimensions -remove GPS antenna -add power to the SMA connector for external GPS antenna -move debug pins -replace ble smd antenna with pсb antenna
Parts:
- removed A1: GGBLA.01.A, RF:GGBLA.01.A, symbol Device:GGBLA.01.A
- removed AE1: AH316M245001-T, AH316M245001-T:XDCR_AH316M245001-T, symbol AH316M245001-T:AH316M245001-T
- removed C31: 22, Capacitor_SMD:C_0402_1005Metric, symbol Device:C
- removed C32: 0.5, Capacitor_SMD:C_0402_1005Metric, symbol Device:C
- removed C33: 0.8, Capacitor_SMD:C_0402_1005Metric, symbol Device:C
- removed C34: 2.7, Capacitor_SMD:C_0402_1005Metric, symbol Device:C
- removed C35: NC, Capacitor_SMD:C_0402_1005Metric, symbol Device:C
- removed C40: 1, Capacitor_SMD:C_0201_0603Metric, symbol Device:C
- removed D1, D2, D3, D4: LED, LED_SMD:LED_0603_1608Metric, symbol Device:LED
- removed L7: 3.6nH, Inductor_SMD:L_0402_1005Metric, symbol Device:L
- removed R5: 10k, Resistor_SMD:R_0201_0603Metric, symbol Device:R
- removed R6, R7, R8, R9: 510, Resistor_SMD:R_0201_0603Metric, symbol Device:R
- removed S1: PTS526_SM08_SMTR2_LFS, PTS526_SM08_SMTR2_LFS:SW_PTS526_SM08_SMTR2_LFS, symbol PTS526_SM08_SMTR2_LFS:PTS526_SM08_SMTR2_LFS
- removed TP10: NRF_GPIO_03, TestPoint:TestPoint_Pad_D2.0mm, symbol Connector:TestPoint
- removed TP11: NRF_GPIO_04, TestPoint:TestPoint_Pad_D2.0mm, symbol Connector:TestPoint
- removed TP12: A9G_GPIO_01, TestPoint:TestPoint_Pad_D2.0mm, symbol Connector:TestPoint
- removed TP8: NRF_GPIO_01, TestPoint:TestPoint_Pad_D2.0mm, symbol Connector:TestPoint
- removed TP9: NRF_GPIO_02, TestPoint:TestPoint_Pad_D2.0mm, symbol Connector:TestPoint
Connections:
- net A9G_GPS_ANT: now also J3.2
Other:
- moved on the sheet: C41, J2, J3, TP13, TP14

Commit message: feat(board): installation GPS antenna, power switch, tag-connect on PCB
Parts:
- removed J2, J3: U.FL-R-SMT-1_10_, U.FL-R-SMT-1_10_:HRS_U.FL-R-SMT-1_10_, symbol U.FL-R-SMT-1_10_:U.FL-R-SMT-1_10_
- removed TP1: +3.3v, TestPoint:TestPoint_Pad_D2.0mm, symbol Connector:TestPoint
- removed TP13: A9G_UART_HST_RX, TestPoint:TestPoint_Pad_D2.0mm, symbol Connector:TestPoint
- removed TP14: A9G_UART_HST_TX, TestPoint:TestPoint_Pad_D2.0mm, symbol Connector:TestPoint
- removed TP17, TP18: SWITCH_BATT+, TestPoint:TestPoint_THTPad_D2.0mm_Drill1.0mm, symbol Connector:TestPoint
- removed TP2: reset, TestPoint:TestPoint_Pad_D2.0mm, symbol Connector:TestPoint
- removed TP3: swdio, TestPoint:TestPoint_Pad_D2.0mm, symbol Connector:TestPoint
- removed TP4: swclk, TestPoint:TestPoint_Pad_D2.0mm, symbol Connector:TestPoint
- removed TP5: gnd, TestPoint:TestPoint_Pad_D2.0mm, symbol Connector:TestPoint
- added C31: 0.1u, Capacitor_SMD:C_0201_0603Metric, symbol Device:C
- added C32: 47, Capacitor_SMD:C_0201_0603Metric, symbol Device:C
- added J5, J6: TC2050-IDC, CONN_TC2050-IDC_TGC, symbol TAG_CONNECT_2050:TC2050-IDC
- added S1: SLW-108645-4A-RA-D, SLW-108645-4A-RA-D:SW_SLW-108645-4A-RA-D, symbol SLW-108645-4A-RA-D:SLW-108645-4A-RA-D
- added U5: SGGP.12.4.A.02, SGGP.12.4.A.02:SGGP.12.4.A.02, symbol SGGP.12.4.A.02:SGGP.12.4.A.02
- added U6: BGU8019, BGU8019:SOT1232, symbol BGU8019:BGU8019
- added U7: ADP150ACBZ-2.8-R7, CB_4_3_ADI, symbol ADP150ACBZ-2.8-R7:ADP150ACBZ-2.8-R7
Connections:
- net +3.3V: now also J5.1
- net +4V: now also S1.3, S1.6, U7.A1 (VIN), U7.B1 (EN)
- net +BATT: now also S1.2, S1.5
- net A9G_GPS_ANT: now also C32.2
- net GND: now also C31.2, J5.3, J5.5, J5.9, J6.3, J6.5, J6.9, S1.7 (SH1), S1.8 (SH2), U5.GND1 (1), U5.GND2 (2), U5.GND3 (3), U5.GND4 (4), U5.GND5 (5), U5.GND6 (6), U5.GND7 (7), U5.GND9 (9), U6.1, U6.4, U7.B2 (GND)
- net HST_RXD: now also J6.8
- net HST_TXD: now also J6.7
- net NRF_RESET: now also J5.10
- net NRF_SWDCLK: now also J5.4
- net NRF_SWDIO: now also J5.2
- new net: U5.RF (8), U6.5
- new net: C32.1, U6.3
- new net +2.8V: C31.1, U6.2, U6.6, U7.A2 (VOUT)
- new net NRF_SWO: J5.6
Other:
- moved on the sheet: TP15, TP16
